Commit message: temp

File: urdf/saber_d6x.urdf (robot description, URDF)
Before this commit: robot saber_d6x, 7 links, 6 joints
Links:
- link base_link: geometry collision mesh filename=package://hex_ros_ik_saber_d6x/urdf/meshes/base_link.STL; visual mesh filename=package://hex_ros_ik_saber_d6x/urdf/meshes/base_link.STL
- link link_1: geometry collision mesh filename=package://hex_ros_ik_saber_d6x/urdf/meshes/link_1.STL; visual mesh filename=package://hex_ros_ik_saber_d6x/urdf/meshes/link_1.STL
- link link_2: geometry collision mesh filename=package://hex_ros_ik_saber_d6x/urdf/meshes/link_2.STL; visual mesh filename=package://hex_ros_ik_saber_d6x/urdf/meshes/link_2.STL
- link link_3: geometry collision mesh filename=package://hex_ros_ik_saber_d6x/urdf/meshes/link_3.STL; visual mesh filename=package://hex_ros_ik_saber_d6x/urdf/meshes/link_3.STL
- link link_4: geometry collision mesh filename=package://hex_ros_ik_saber_d6x/urdf/meshes/link_4.STL; visual mesh filename=package://hex_ros_ik_saber_d6x/urdf/meshes/link_4.STL
- link link_5: geometry collision mesh filename=package://hex_ros_ik_saber_d6x/urdf/meshes/link_5.STL; visual mesh filename=package://hex_ros_ik_saber_d6x/urdf/meshes/link_5.STL
- link link_6: geometry collision mesh filename=package://hex_ros_ik_saber_d6x/urdf/meshes/link_6.STL; visual mesh filename=package://hex_ros_ik_saber_d6x/urdf/meshes/link_6.STL
